Commit message: urdf working

File: actual_arm_urdf.urdf (robot description, URDF)
Before this commit: robot robotic_arm, 6 links, 5 joints
Links:
- link base_link: mass None -> 1.0; geometry collision cylinder length=0.09 radius=0.15; visual cylinder length=0.09 radius=0.15
- link base_rot: mass None -> 0.5; geometry collision box size=0.07 0.078 0.052; visual box size=0.07 0.078 0.052
- link center_arm: mass None -> 0.3; geometry collision cylinder length=0.1725 radius=0.055; visual cylinder length=0.1725 radius=0.055
- link gripper: mass None -> 0.1; geometry collision box size=0.2 0.05 0.025; visual box size=0.2 0.05 0.025
- link lower_arm: mass None -> 0.4; geometry collision cylinder length=0.2475 radius=0.07; visual cylinder length=0.2475 radius=0.07
- link upper_arm: mass None -> 0.2; geometry collision cylinder length=0.1075 radius=0.05; visual cylinder length=0.1075 radius=0.05
Joints:
- joint elbow_joint: origin xyz=0 0 0.2475 rpy=0 0 0 -> xyz=0 0 0.2475
- joint shoulder_joint: origin xyz=0 0 0.026 rpy=0 0 0 -> xyz=0 0 0.026
- joint wrist_joint_1: origin xyz=0 0 0.1725 rpy=0 0 0 -> xyz=0 0 0.1725
- joint wrist_joint_2: origin xyz=0 0 0.1075 rpy=0 0 0 -> xyz=0 0 0.1075
